File: md_test_v1/moterdriver_test_v1.kicad_sch (KiCad schematic)
At the start: 20 parts, among them J1 Conn_01x02_Socket, J2 Conn_01x03_Socket, J3 Conn_01x02_Socket, Q1 rs6, Q2 rs6, Q3 rs6, Q4 rs6, U1 DRV8701PRGER

Commit message: md改良(ちょっと前にしたやつ上げ忘れ)
Parts:
- removed J2: Conn_01x03_Socket, Connector_JST:JST_XH_S3B-XH-A_1x03_P2.50mm_Horizontal, symbol Connector:Conn_01x03_Socket
- removed Q1, Q2, Q3, Q4: rs6, Package_SO:PowerPAK_SO-8_Single, symbol Transistor_FET:SiR696DP
- removed R1: 10k, Resistor_SMD:R_0603_1608Metric_Pad0.98x0.95mm_HandSolder, symbol Device:R_Small
- added C10, C9: 10uF, Capacitor_SMD:C_0805_2012Metric_Pad1.18x1.45mm_HandSolder, symbol Device:C_Small
- added C8: 250uF, Capacitor_THT:CP_Radial_D5.0mm_P2.50mm, symbol Device:C
- added D1: D_TVS, symbol Device:D_TVS
- added J4: Conn_02x06_Odd_Even, Connector_PinHeader_2.54mm:PinHeader_2x06_P2.54mm_Vertical, symbol Connector_Generic:Conn_02x06_Odd_Even
- added Q1, Q2, Q3, Q4: Q_NMOS_GDS, Package_TO_SOT_SMD:TO-252-2, symbol Transistor_FET:Q_NMOS_GDS
- added R10, R11, R6, R7, R8, R9: 10k, Resistor_SMD:R_0603_1608Metric_Pad0.98x0.95mm_HandSolder, symbol Device:R_Small
- added R12: 1k, Resistor_SMD:R_0603_1608Metric_Pad0.98x0.95mm_HandSolder, symbol Device:R_Small
- C1, C2: value 0.1uf -> 1uF
- R2: value 70k -> 18k
- R3: value 75k -> 200k
- R5: value 10mi -> 2m
Connections:
- net +24V: now also C10.1, C8.2, C9.1, D1.1 (A1), Q2.2 (D), Q4.2 (D)
- net GND1: now also C10.2, C8.1, C9.2, D1.2 (A2), J4.1 (Pin_1), J4.11 (Pin_11), J4.3 (Pin_3), J4.5 (Pin_5), J4.7 (Pin_7), J4.9 (Pin_9)
- net SO_out: now also R12.1
- net faultN_out: now also J4.8 (Pin_8), R6.1
- net pwm_in1: now also J4.2 (Pin_2)
- net pwm_in2: now also J4.4 (Pin_4)
- net sleepN_in: now also J4.6 (Pin_6)
- net sns_out: now also J4.10 (Pin_10), R7.1
- net at J3.2 (Pin_2), U1.18 (SH1): now also Q3.2 (D), Q4.3 (S), R8.1
- net at U1.17 (GH1): now also Q4.1 (G), R8.2
- net at C2.1, U1.8 (DVDD): now also R6.2, R7.2
- net at U1.19 (GL1): now also Q3.1 (G), R9.1
- net at R5.1, U1.21 (SP): now also Q1.3 (S), Q3.3 (S), R11.1, R9.2
- net at U1.22 (GL2): now also Q1.1 (G), R11.2
- net at J3.1 (Pin_1), U1.23 (SH2): now also Q1.2 (D), Q2.3 (S), R10.1
- net at U1.24 (GH2): now also Q2.1 (G), R10.2
- new net: J4.12 (Pin_12), R12.2
Other:
- note added: "XT60"
- note added: "source"
- note removed: "sorce"
- moved on the sheet: C2, C3, C4, C5, J1, R5

Commit message: MDを設計した(できたと思っている)
Parts:
- added D3: D_Zener, Diode_SMD:D_SOD-123, symbol Device:D_Zener
- added Q5, Q6: Q_NMOS_GDS, Package_TO_SOT_SMD:TO-252-2, symbol Transistor_FET:Q_NMOS_GDS
- added R13: 10k, Resistor_SMD:R_0603_1608Metric_Pad0.98x0.95mm_HandSolder, symbol Device:R_Small
- C8: footprint Capacitor_THT:CP_Radial_D5.0mm_P2.50mm -> Capacitor_THT:CP_Radial_D12.5mm_P5.00mm
- D1: footprint (none) -> Diode_SMD:D_SMB
- R5: footprint Resistor_SMD:R_2816_7142Metric_Pad3.20x4.45mm_HandSolder -> Resistor_SMD:R_1225_3264Metric_Pad1.47x6.45mm_HandSolder
- U1: footprint drv8701prger:RGE0024F -> drv8701:RGE0024F
Connections:
- net +24V: now also C8.1, R13.1; no longer C8.2
- net GND1: now also C8.2, J4.10 (Pin_10), J4.12 (Pin_12), J4.2 (Pin_2), J4.4 (Pin_4), J4.6 (Pin_6), J4.8 (Pin_8), D3.2 (A), Q5.2 (D), Q6.2 (D); no longer C8.1, J1.1 (Pin_1), J4.1 (Pin_1), J4.11 (Pin_11), J4.3 (Pin_3), J4.5 (Pin_5), J4.7 (Pin_7), J4.9 (Pin_9)
- net faultN_out: now also J4.7 (Pin_7); no longer J4.8 (Pin_8)
- net pwm_in1: now also J4.1 (Pin_1); no longer J4.2 (Pin_2)
- net pwm_in2: now also J4.3 (Pin_3); no longer J4.4 (Pin_4)
- net sleepN_in: now also J4.5 (Pin_5); no longer J4.6 (Pin_6)
- net sns_out: now also J4.9 (Pin_9); no longer J4.10 (Pin_10)
- net at R12.2: now also J4.11 (Pin_11); no longer J4.12 (Pin_12)
- new net: D3.1 (K), Q5.1 (G), Q6.1 (G), R13.2
- new net GND: J1.1 (Pin_1), Q5.3 (S), Q6.3 (S)
Other:
- note added: "定格50V以上厳守"
- moved on the sheet: J1

Commit message: 電源基板の追加
Parts:
- removed D1: D_TVS, Diode_SMD:D_SMB, symbol Device:D_TVS
- added D2: SMBJ26A, Diode_SMD:D_SMB, symbol Diode:SM6T27A
- added R14, R15: 10, Resistor_SMD:R_0603_1608Metric_Pad0.98x0.95mm_HandSolder, symbol Device:R_Small
Connections:
- net +24V: now also D2.1 (A1)
- net GND: now also Q5.2 (D), Q6.2 (D); no longer Q5.3 (S), Q6.3 (S)
- net GND1: now also Q5.3 (S), Q6.3 (S), D2.2 (A2); no longer Q5.2 (D), Q6.2 (D)
- net at D3.1 (K), R13.2: now also R14.1, R15.1; no longer Q5.1 (G), Q6.1 (G)
- new net: Q5.1 (G), R15.2
- new net: Q6.1 (G), R14.2
Other:
- moved on the sheet: Q5

Commit message: MDのGND経路の微修正
Connections:
- net faultN_out: now also J4.9 (Pin_9); no longer J4.7 (Pin_7)
- net sns_out: now also J4.7 (Pin_7); no longer J4.9 (Pin_9)
Changed lines of the file:
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@@
+	(wire
+		(pts
+			(xy 99.06 114.3) (xy 113.03 114.3)
+		)
+		(stroke
+			(width 0)
+			(type default)
+		)
+	)
 	(wire
 		(pts
@@
 	(wire
 		(pts
-			(xy 110.49 114.3) (xy 110.49 124.46)
+			(xy 110.49 111.76) (xy 110.49 124.46)
 		)
 		(stroke
@@
 	(wire
 		(pts
+			(xy 110.49 111.76) (xy 99.06 111.76)
+		)
+		(stroke
+			(width 0)
+			(type default)
+		)
+	)
+	(wire
+		(pts
 			(xy 190.5 124.46) (xy 204.47 124.46)
 		)
@@
 	(wire
 		(pts
+			(xy 113.03 114.3) (xy 113.03 121.92)
+		)
+		(stroke
+			(width 0)
+			(type default)
+		)
+	)
+	(wire
+		(pts
 			(xy 127 120.65) (xy 127 124.46)
 		)
@@
 	(wire
 		(pts
-			(xy 99.06 111.76) (xy 113.03 111.76)
-		)
-		(stroke
-			(width 0)
-			(type default)
-		)
-	)
-	(wire
-		(pts
 			(xy 228.6 60.96) (xy 246.38 60.96)
 		)
@@
 	(wire
 		(pts
-			(xy 99.06 114.3) (xy 110.49 114.3)
-		)
-		(stroke
-			(width 0)
-			(type default)
-		)
-	)
-	(wire
-		(pts
 			(xy 238.76 128.27) (xy 238.76 129.54)
 		)
@@
 		(pts
 			(xy 228.6 134.62) (xy 228.6 135.89)
-		)
-		(stroke
-			(width 0)
-			(type default)
-		)
-	)
-	(wire
-		(pts
-			(xy 113.03 121.92) (xy 113.03 111.76)
 		)
 		(stroke
@@
 		)
 	)
-	(label "faultN_out"
-		(at 102.87 111.76 0)
-		(effects
-			(font
-				(size 1.27 1.27)
-			)
-			(justify left bottom)
-		)
-	)
 	(label "SO_out"
 		(at 198.12 109.22 0)
@@
 		)
 	)
-	(label "sns_out"
-		(at 102.87 114.3 0)
-		(effects
-			(font
-				(size 1.27 1.27)
-			)
-			(justify left bottom)
-		)
-	)
 	(label "Vref"
 		(at 191.77 111.76 180)
@@
 		)
 	)
+	(label "sns_out"
+		(at 102.87 111.76 0)
+		(effects
+			(font
+				(size 1.27 1.27)
+			)
+			(justify left bottom)
+		)
+	)
 	(label "vm"
 		(at 222.25 95.25 180)
@@
 		)
 	)
+	(label "faultN_out"
+		(at 102.87 114.3 0)
+		(effects
+			(font
+				(size 1.27 1.27)
+			)
+			(justify left bottom)
+		)
+	)
