File: moter_powerup_boardv3/moter_upgrade_boardv1.kicad_sch (KiCad schematic)
At the start: 36 parts, among them J1 Conn_01x05_Socket, J2 Conn_ST_STDC14, J3 Conn_01x02_Socket, J4 Conn_01x02_Socket, J5 Conn_01x02_Socket, J6 Conn_01x03_Pin, Q2 Q_PMOS_GDS, SW1 SW_Wuerth_450301014042, SW2 SW_Push, SW3 SW_Push, SW4 SW_Push, U2 PTCAN3414DDFR, U3 STM32H533CETx

Commit message: MDPID基板を作ったりLED基板の電源回りをいじった
MDPIDの電源変更+配線
LED基板の電源変更(未配線)
Parts:
- removed J3, J4, J5: Conn_01x02_Socket, Connector_JST:JST_XH_S2B-XH-A-1_1x02_P2.50mm_Horizontal, symbol Connector:Conn_01x02_Socket
- removed Q2: Q_PMOS_GDS, Package_TO_SOT_THT:TO-220-3_Horizontal_TabUp, symbol Transistor_FET:Q_PMOS_GDS
- removed R5, R7: 10k, Resistor_SMD:R_0805_2012Metric, symbol Device:R
- removed R8: 100k, Resistor_SMD:R_0805_2012Metric, symbol Device:R
- removed SW2, SW3: SW_Push, Button_Switch_THT:SW_PUSH_6mm, symbol Switch:SW_Push
- added C11, C14: 4.7uF, Capacitor_SMD:C_0603_1608Metric_Pad1.08x0.95mm_HandSolder, symbol Device:C_Small
- added C12: 10nF, Capacitor_SMD:C_0603_1608Metric_Pad1.08x0.95mm_HandSolder, symbol Device:C_Small
- added C15: 220uF, Capacitor_SMD:CP_Elec_6.3x4.5, symbol Device:C_Polarized_Small
- added D3, D4: D_Shockley, Diode_SMD:D_SMB, symbol Device:D_Shockley
- added J3, J5: Conn_01x03_Pin, Connector_JST:JST_XH_S3B-XH-A_1x03_P2.50mm_Horizontal, symbol Connector:Conn_01x03_Pin
- added J7: Conn_01x02_Socket, Connector_JST:JST_XH_S2B-XH-A-1_1x02_P2.50mm_Horizontal, symbol Connector:Conn_01x02_Socket
- added L1: 22uH, Inductor_SMD:L_6.3x6.3_H3, symbol Device:L
- added R6: 10k, Resistor_SMD:R_0603_1608Metric_Pad0.98x0.95mm_HandSolder, symbol Device:R_Small
- added R7: 5.90k, Resistor_SMD:R_0603_1608Metric_Pad0.98x0.95mm_HandSolder, symbol Device:R_Small
- added U3: TPS5430DDA, Package_SO:TI_SO-PowerPAD-8_ThermalVias, symbol Regulator_Switching:TPS5430DDA
- J6: footprint TerminalBlock_RND:TerminalBlock_RND_205-00233_1x03_P5.08mm_Horizontal -> Connector_JST:JST_XH_S3B-XH-A-1_1x03_P2.50mm_Horizontal
- U1: renamed from U2; footprint 26off_tcan3414ddfr:SOT-23-THIN-8_DDF_TEX -> 26off_tcan3414ddfr:SOT-23-THIN-8_DDF_TEX-M
- renumbered C7 to C1, C8 to C10, C6 to C2, C5 to C3, C12 to C4, C11 to C5, C9 to C6, C1 to C7, C2 to C8, C3 to C9, R6 to R3, R2 to R4, R3 to R5, SW4 to SW2, U3 to U2
Connections:
- net dir to moter is gone; now on net PWM1: J6.1 (Pin_1)
- net mb is gone; now on an unnamed net: U2.3 (PC14)
- net pwm to moter is gone; now on net PWM2: J6.2 (Pin_2)
- net +3.3V: now also U2.9 (VDDA), C15.1, L1.2, R6.1
- net CAN1R: now also SW1.1 (B); no longer SW1.2 (C)
- net CAN1_+: now also SW1.2 (C), J3.2 (Pin_2), J5.2 (Pin_2)
- net CAN1_-: now also J3.3 (Pin_3), J5.1 (Pin_1); no longer SW1.1 (B)
- net GND: now also C11.2, C14.2, C15.2, D3.2 (A), J3.1 (Pin_1), J5.3 (Pin_3), J7.1 (Pin_1), R7.2, U3.6 (GND), U3.9 (GNDPAD)
- net en-a: now also J1.1 (Pin_1); no longer J1.3 (Pin_3)
- net en-b: now also J1.3 (Pin_3); no longer J1.1 (Pin_1)
- net at D1.2 (A): no longer U2.6 (PH1)
- new net: D4.2 (A), J7.2 (Pin_2)
- new net: C12.1, U3.1 (BOOT)
- new net: R6.2, R7.1, U3.4 (VSENSE)
- new net: C12.2, D3.1 (K), L1.1, U3.8 (PH)
- new net +24V: C11.1, C14.1, D4.1 (K), U3.7 (VIN)
Other:
- moved on the sheet: C10, C6, C7, C8, C9
